File: ESR_Meter_Develop_RevA/ESR_Meter_Develop_RevA.kicad_sch (KiCad schematic)
At the start: 0 parts

Commit message: WIP
Changed lines of the file:
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@@
 	(generator_version "9.0")
 	(paper "A4")
+	(text_box "+/- 14V Boost"
+		(exclude_from_sim no)
+		(at 152.4 57.15 0)
+		(size 10.16 5.08)
+		(margins 0.9525 0.9525 0.9525 0.9525)
+		(stroke
+			(width 0)
+			(type solid)
+		)
+		(fill
+			(type color)
+			(color 142 238 255 1)
+		)
+		(effects
+			(font
+				(size 0.889 0.889)
+			)
+		)
+	)
+	(text_box "+3V BUCK"
+		(exclude_from_sim no)
+		(at 152.4 50.8 0)
+		(size 10.16 3.81)
+		(margins 0.9525 0.9525 0.9525 0.9525)
+		(stroke
+			(width 0)
+			(type solid)
+		)
+		(fill
+			(type color)
+			(color 142 238 255 1)
+		)
+		(effects
+			(font
+				(size 0.889 0.889)
+			)
+		)
+	)
+	(text_box "+2.5V LDO"
+		(exclude_from_sim no)
+		(at 167.64 50.8 0)
+		(size 10.16 3.81)
+		(margins 0.9525 0.9525 0.9525 0.9525)
+		(stroke
+			(width 0)
+			(type solid)
+		)
+		(fill
+			(type color)
+			(color 142 238 255 1)
+		)
+		(effects
+			(font
+				(size 0.889 0.889)
+			)
+		)
+	)
 	(sheet
 		(at 38.1 63.5)

Commit message: backup WIP
Other:
- added sheet Backend (backend.kicad_sch)
Changed lines of the file:
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@@
+	)
+	(sheet
+		(at 38.1 74.93)
+		(size 12.7 3.81)
+		(exclude_from_sim no)
+		(in_bom yes)
+		(on_board yes)
+		(dnp no)
+		(fields_autoplaced yes)
+		(stroke
+			(width 0.1524)
+			(type solid)
+		)
+		(fill
+			(color 255 255 255 0.0000)
+		)
+		(property "Sheetname" "Backend"
+			(at 38.1 74.2184 0)
+			(effects
+				(font
+					(size 1.27 1.27)
+				)
+				(justify left bottom)
+			)
+		)
+		(property "Sheetfile" "backend.kicad_sch"
+			(at 38.1 79.3246 0)
+			(effects
+				(font
+					(size 1.27 1.27)
+				)
+				(justify left top)
+			)
+		)
+		(instances
+			(project "ESR_Meter_Develop_RevA"
+				(path "/9db92e0e-011b-43dc-aa19-665c004a2f0f"
+					(page "3")
+				)
+			)
+		)
 	)
 	(sheet

Commit message: bckp
Other:
- added sheet Power Supply (power_supply.kicad_sch)
Changed lines of the file:
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@@
+		)
+	)
+	(sheet
+		(at 38.1 86.36)
+		(size 12.7 3.81)
+		(exclude_from_sim no)
+		(in_bom yes)
+		(on_board yes)
+		(dnp no)
+		(fields_autoplaced yes)
+		(stroke
+			(width 0.1524)
+			(type solid)
+		)
+		(fill
+			(color 255 255 255 0.0000)
+		)
+		(property "Sheetname" "Power Supply"
+			(at 38.1 85.6484 0)
+			(effects
+				(font
+					(size 1.27 1.27)
+				)
+				(justify left bottom)
+			)
+		)
+		(property "Sheetfile" "power_supply.kicad_sch"
+			(at 38.1 90.7546 0)
+			(effects
+				(font
+					(size 1.27 1.27)
+				)
+				(justify left top)
+			)
+		)
+		(instances
+			(project "ESR_Meter_Develop_RevA"
+				(path "/9db92e0e-011b-43dc-aa19-665c004a2f0f"
+					(page "4")
+				)
+			)
 		)
 	)
