File: ESR_Meter_Develop_RevA/esr_frontend.kicad_sch (KiCad schematic)
At the start: 23 parts, among them U1 TL074HIDR

Commit message: working on frontend
Parts:
- added C6: 22nF 2kV, 3Brain_Capacitors:C_1812, symbol 3Brain_Capacitors:N_22nF_2kV_1812
- added D6: BAV99, 3Brain_Diodes:SOT-23_ACAC, symbol 3Brain_Diodes:BAV99
- added D7, D8: M1, 3Brain_Diodes:D_SMA, symbol 3Brain_Diodes:M1
- added D9: SD12C-01FTG, 3Brain_Diodes:D_SOD-323_Bipolar, symbol 3Brain_Diodes:SD12C TVS
- added K1: 1462038-4, 3Brain_Miscellaneous:AXICOM_Relay_IM, symbol 3Brain_Miscellaneous:Relay_1462038-4
- added R13: 2.2k, 3Brain_Resistors:R_1210, symbol 3Brain_Resistors:_template_1210_duplicate_me
- added R14: 1k, 3Brain_Resistors:R_0603, symbol 3Brain_Resistors:K_1k_0603
- added R15: 220R, 3Brain_Resistors:R_0603, symbol 3Brain_Resistors:R_220R_0603
- added R16: 1k, 3Brain_Resistors:R_Axial__L17.0mm_D6.0mm_P25.40mm_H, symbol 3Brain_Resistors:R_Small
- added R17: 100R, 3Brain_Resistors:R_1210, symbol 3Brain_Resistors:_template_1210_duplicate_me
- added RTH1: 1k, 3Brain_Miscellaneous:PTCEL13, symbol 3Brain_Miscellaneous:PTC_1k
- added U2: TL071H, 3Brain_ICs:SOIC-8, symbol 3Brain_AnalogIC:TL071H
Connections:
- net GND: now also D7.A, D8.C
- net at D1.C, D2.A, R5.1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: now also R13.2
- net VSS: now reaches C3.2, U1.11 (V-)
- net VSS: now also U2.4 (V-)
- net at R3.1: now also C6.1, K1.3, K1.6
- net VDD: now reaches C2.1, U1.4 (V+)
- net VDD: now also U2.7 (V+)
- new net: K1.2, K1.7, R16.1
- new net: K1.4, K1.5, R17.1
- new net: D7.C, D8.A, R14.1, R15.1, R17.2, RTH1.1
- new net: D9.A1, K1.8
- new net: D9.A2, K1.1 (+)
- new net: R16.2, RTH1.2
- new net: D6.AC, R14.2, U2.2 (-)
- new net: D6.A, D6.C, R15.2, U2.6
- new net: C6.2, R13.1
Other:
- moved on the sheet: C1, R1, R2, R3, R4

Commit message: WIP
Parts:
- added C7: 100pF, 3Brain_Capacitors:C_0603, symbol 3Brain_Capacitors:_template_0603_duplicate_me
- added R18: 18k, 3Brain_Resistors:R_0603, symbol 3Brain_Resistors:_template_0603_duplicate_me
- added R19: 2k, 3Brain_Resistors:R_0603, symbol 3Brain_Resistors:_template_0603_duplicate_me
Connections:
- net GND: now also C7.2, R19.2
- net at U2.3 (+): now also R18.1
- new net SINE_DAC: C7.1, R18.2, R19.1

Commit message: bckp
Parts:
- added C10, C11, C12, C9: 100nF, 3Brain_Capacitors:C_0603, symbol 3Brain_Capacitors:N_100nF_50V_0603
- added C8: 1uF, 3Brain_Capacitors:C_0603, symbol 3Brain_Capacitors:U_1uF_50V_0603
- added R20, R21, R22, R23: 10k, 3Brain_Resistors:R_0603, symbol 3Brain_Resistors:K_10k_0603
- added U3: TL072H, 3Brain_ICs:SOIC-8, symbol 3Brain_AnalogIC:TL072H
Connections:
- net +2.5V: now also R21.1
- net GND: now also C10.1, C11.2, C12.1, C9.2
- net SINE_DAC: now also C8.2; no longer C7.1, R18.2, R19.1
- net VDD: now also C11.1, C9.1, U3.8 (V+)
- net VSS: now also C10.2, C12.2, U3.4 (V-)
- net at C1.1, R1.2, R4.1: now also U3.3 (+)
- net at C5.1, D5.A, R12.2: now also R23.1
- new net: C7.1, C8.1, R18.2, R19.1
- new net: R20.1, U3.1, U3.2 (-)
- new net: R20.2, R21.2, U3.5 (+)
- new net: R22.1, U3.6 (-), U3.7
- new net ESR_ADC: R23.2
- new net V_MEAS_ADC: R22.2
Other:
- moved on the sheet: C1, C5, C7, D5, D6, D7, D8, K1B, K1C, R1, R12, R14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

Commit message: bckp
Parts:
- removed C10, C9: 100nF, 3Brain_Capacitors:C_0603, symbol 3Brain_Capacitors:N_100nF_50V_0603
- removed U2: TL071H, 3Brain_ICs:SOIC-8, symbol 3Brain_AnalogIC:TL071H
- removed U3: TL072H, 3Brain_ICs:SOIC-8, symbol 3Brain_AnalogIC:TL072H
- added U2: TL074HIDR, 3Brain_ICs:SOIC-14, symbol 3Brain_AnalogIC:TL074H
Connections:
- net SINE_DAC: now also U2.5 (+); no longer C8.2
- net VDD: now also U2.4 (V+)
- net VSS: now also U2.11 (V-)
- net at R18.1: now also C7.1, R19.1, U2.3 (+)
- net at C8.1, R18.2: no longer C7.1, R19.1
- net at C1.1, R1.2, R4.1: now also U2.10 (+)
- net at D6.AC, R14.2: now also U2.2 (-)
- net at D6.A, D6.C, R15.2: now also U2.1
- net at R20.1: now also U2.8, U2.9 (-)
- net at R20.2, R21.2: now also U2.12 (+)
- net at R22.1: now also U2.13 (-), U2.14
- new net: C8.2, U2.6 (-), U2.7
Other:
- moved on the sheet: C1, C11, C12, C2, C3, C4, C5, C6, C7, C8, D1, D2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

Commit message: backup WIP
Parts:
- added Q1: DMN62D0, 3Brain_Transistors:SOT-23_GSD, symbol 3Brain_Transistors:DMN62D0U-7
- added R24: 10k, 3Brain_Resistors:R_0603, symbol 3Brain_Resistors:K_10k_0603
- added unit 3 of U2
- added unit 4 of U2
- added unit 1 of U2
- added unit 2 of U2
Connections:
- net GND: now also Q1.S, R24.1
- net SINE_DAC: now also U2.5 (+); no longer U2.5 (+)
- net at C7.1, R18.1, R19.1: now also U2.3 (+); no longer U2.3 (+)
- net at D9.A1, K1.8: now also Q1.D
- net +3.0V: now reaches D9.A2, K1.1 (+)
- net at C1.1, R1.2, R4.1: now also U2.10 (+); no longer U2.10 (+)
- net at D6.A, D6.C, R15.2: now also U2.1; no longer U2.1
- net at R20.2, R21.2: now also U2.12 (+); no longer U2.12 (+)
- net at D6.AC, R14.2: now also U2.2 (-); no longer U2.2 (-)
- new net: R20.1, U2.8, U2.9 (-)
- new net: R22.1, U2.13 (-), U2.14
- new net: C8.2, U2.6 (-), U2.7
- new net RELAY: Q1.G, R24.2
Other:
- moved on the sheet: C1, C11, C12, C2, C3, C4, C5, C6, C7, C8, D1, D2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

Commit message: bckp
Other:
- note added: "Try TL064"
- moved on the sheet: C11, C12, C2, C3, D7, D9, K1A, Q1, R24, U1E, U2E
